File: tiristoriaus_plokste.sch (KiCad schematic (older format))
At the start: 39 parts, among them X1 Faston_6.3x08x14, X2 Faston_6.3x08x14, X3 Faston_6.3x08x14

Commit message: plokstes dviem tiristoriams projektavimas. gerber failu ruosimas gamybai
Parts:
- removed R1, R? (x2): 330R, resistors:R_1206, symbol R_330R_1206_1%
- removed R? (x2): LOAD1.1, resistors:R_Axial_DIN0411_L9.9mm_D3.6mm_P15.24mm_Horizontal, symbol R_0R22_2W_5%
- removed R? (x2): LOAD1.2, resistors:R_Axial_DIN0411_L9.9mm_D3.6mm_P15.24mm_Horizontal, symbol R_0R22_2W_5%
- removed R? (x2): LOAD3.1, resistors:R_Axial_DIN0411_L9.9mm_D3.6mm_P15.24mm_Horizontal, symbol R_0R22_2W_5%
- removed R? (x2): LOAD3.2, resistors:R_Axial_DIN0411_L9.9mm_D3.6mm_P15.24mm_Horizontal, symbol R_0R22_2W_5%
- removed R? (x2): LOAD2.2, resistors:R_Axial_DIN0411_L9.9mm_D3.6mm_P15.24mm_Horizontal, symbol R_0R22_2W_5%
- removed R? (x2): LOAD2.1, resistors:R_Axial_DIN0411_L9.9mm_D3.6mm_P15.24mm_Horizontal, symbol R_0R22_2W_5%
- added D1 (x4): BTW67, symbol disc:Q_BTW67
- added D? (x4): LL4007, symbol disc:D_LL4007
- added LOAD1.1 (x2), LOAD1.2 (x2), LOAD2.1 (x2), LOAD2.2 (x2), LOAD3.1 (x2), LOAD3.2 (x2): Heater, symbol Device:Heater
- added R1: 470R, resistors:R_1206, symbol resistors_us:R_470R_1206_1%
- added R? (x4): 1k, symbol resistors_us:R_1k_1206_1%
- added R? (x8): 470R, symbol resistors_us:R_470R_1206_1%
- added R? (x4): 330, symbol resistors_us:R_1k_1206_1%
- added U? (x2): MOC3060S, symbol disc:MOC3060S
- added X4: Faston_6.3x08x14, mech:Faston_6.3x0.8x14, symbol mech:Faston_6.3x08x14
- D1: symbol Q_BTW67 -> disc:Q_BTW67
- D10, D13, D14, D3, D4, D5, D8, D9: renamed from D?; symbol TRIAC -> various:TRIAC
- D11: renamed from D?; value TRIAC 2 -> Q2; symbol TRIAC -> various:TRIAC
- D12: renamed from D?; value TRIAC 4 -> Q4; symbol TRIAC -> various:TRIAC
- D2: symbol D_LL4007 -> disc:D_LL4007
- D6: renamed from D?; value TRIAC 1 -> Q1; symbol TRIAC -> various:TRIAC
- D7: renamed from D?; value TRIAC 3 -> Q3; symbol TRIAC -> various:TRIAC
- R13, R18, R20, R3: renamed from R?; symbol R_0R22_2W_5% -> resistors_us:R_0R22_2W_5%
- R2: symbol R_1k_1206_1% -> resistors_us:R_1k_1206_1%
- U1, U2: renamed from U?; symbol MOC3060S -> disc:MOC3060S
- X1: value Faston_6.3x08x14 -> A; symbol Faston_6.3x08x14 -> mech:Faston_6.3x08x14
- X2: symbol Faston_6.3x08x14 -> mech:Faston_6.3x08x14
- X3: value Faston_6.3x08x14 -> K; symbol Faston_6.3x08x14 -> mech:Faston_6.3x08x14
Connections:
- net labels added: FAZE1, FAZE3, LOAD1, LOAD3, X1, X12, X14, X17, X2, X26, X3, X7, X9
- wire segments 146 -> 224
Other:
- note added: "V1"
- note added: "V2"
- note added: "V3"
- note added: "V4"
- moved on the sheet: D1, D2, R2, X1, X2, X3
