File: tiristoriaus_plokste/x2/tp_x2.sch (KiCad schematic (older format))
At the start: 78 parts, among them U1 MOC3060S, U2 MOC3060S, X1 LD3, X10 Faston_6.3x08x14, X11 Faston_6.3x08x14, X12 Faston_6.3x08x14, X13 Faston_6.3x08x14, X14 Faston_6.3x08x14, X17 Faston_6.3x08x14, X2 PH3, X26 Faston_6.3x08x14, X3 Faston_6.3x08x14, X4 LD1, X5 PH1, X6 Faston_6.3x08x14, X7 Faston_6.3x08x14, X8 Faston_6.3x08x14, X9 Faston_6.3x08x14

Commit message: sugeneruoti nauji gerberiai, paruostos principine ir surinkimo schemos.
Parts:
- removed H10, H11, H12, H13, H14, H15, H16, H17, H18, H19, H20, H22, H23, H24, H27, H28, H29, H30, H31, H32, H33, H34, H35, H36, H37, H38, H39, H40, H5, H6, H9: Conn_01x01, Wire_Pads:SolderWirePad_single_1mmDrill, symbol Connector_Generic:Conn_01x01
- removed RV1, RV3: 480V, disc:VR_VE420V, symbol Device:Varistor_US
- removed X10, X3, X6, X8: Faston_6.3x08x14, mech:Faston_6.3x0.8x14, symbol mech:Faston_6.3x08x14
- added H4: Conn_01x01, Wire_Pads:SolderWirePad_single_1mmDrill, symbol Connector_Generic:Conn_01x01
- added T1: Transformer_1P_1S, symbol Device:Transformer_1P_1S
- V1.1, V1.2, V2.1, V2.2: ventcode - -> ZELT046
- X1: value LD3 -> LD1
- X2: value PH3 -> PH1
- X4: value LD1 -> LD3
- X5: value PH1 -> PH3
- renumbered X13 to X3, X11 to X6
Connections:
- net labels added: EKR_PH1, EKR_PH3
- wire segments 175 -> 106

Commit message: paskutinis variantas. sugeneruoti nauji gerberiai
Parts:
- renumbered V1.2 to V1.1, V1.1 to V1.2, V2.2 to V2.1, V2.1 to V2.2
Changed lines of the file:
@@
 $EndDescr
 $Comp
-L disc:Q_BTW67 V2.2
+L disc:Q_BTW67 V2.1
 U 1 1 5BE35DAB
 P 7000 3950
-F 0 "V2.2" H 6750 4100 50  0000 L CNN
+F 0 "V2.1" H 6750 4100 50  0000 L CNN
 F 1 "BTW67" H 6700 4000 50  0000 L CNN
 F 2 "disc:RD91" H 7450 4000 50  0001 C CNN
@@
 Connection ~ 6450 4600
 $Comp
-L disc:Q_BTW67 V2.1
+L disc:Q_BTW67 V2.2
 U 1 1 5BBEE31B
 P 7700 4250
-F 0 "V2.1" H 7450 4300 50  0000 L CNN
+F 0 "V2.2" H 7450 4300 50  0000 L CNN
 F 1 "BTW67" H 7350 4400 50  0000 L CNN
 F 2 "disc:RD91" H 8150 4300 50  0001 C CNN
@@
 	3500 4600 3600 4600
 $Comp
-L disc:Q_BTW67 V1.2
+L disc:Q_BTW67 V1.1
 U 1 1 5BC0D088
 P 7000 2500
-F 0 "V1.2" H 6750 2650 50  0000 L CNN
+F 0 "V1.1" H 6750 2650 50  0000 L CNN
 F 1 "BTW67" H 6700 2550 50  0000 L CNN
 F 2 "disc:RD91" H 7450 2550 50  0001 C CNN
@@
 Connection ~ 6450 3150
 $Comp
-L disc:Q_BTW67 V1.1
+L disc:Q_BTW67 V1.2
 U 1 1 5BC0D0F6
 P 7700 2800
-F 0 "V1.1" H 7450 2850 50  0000 L CNN
+F 0 "V1.2" H 7450 2850 50  0000 L CNN
 F 1 "BTW67" H 7350 2950 50  0000 L CNN
 F 2 "disc:RD91" H 8150 2850 50  0001 C CNN

Commit message: 2019-04-28
Parts:
- EKR_X12, EKR_X14, EKR_X17, EKR_X26, EKR_X7, EKR_X9: Aukstis 10 -> (none); Gamintojo Kodas - -> (none); Kaina 0 -> (none); Komentaras - -> (none); Korpusas - -> (none); Korpuso tipas DIP -> (none); Marke - -> (none); Nominalas - -> (none); Nuoroda - -> (none); Parametras - -> (none); Pavadinimas Kontaktas -> (none); ventcode ZAJ023 -> (none)
- R10, R5: Aukstis 1 -> (none); Gamintojo Kodas - -> (none); Kaina 0.001 -> (none); Komentaras - -> (none); Korpusas 1206 -> (none); Korpuso tipas SMD -> (none); Marke - -> (none); Nominalas 470R -> (none); Nuoroda - -> (none); Parametras - -> (none); Pavadinimas Rezistorius -> (none); ventcode - -> (none)
- U1, U2: Gamintojo kodas MOC3060S -> (none); Kaina 0 -> (none); Korpuso tipas SMD -> (none); Pavadinimas Optosimistorius -> (none); ventcode - -> (none)
Changed lines of the file:
@@
 F 2 "" H 3300 2750 50  0001 L CIN
 F 3 "http://datasheet.octopart.com/MOC3063SR2M-Fairchild-Semiconductor-datasheet-10497244.pdf" H 3300 2650 50  0001 L CNN
-F 4 "-" H 2450 2300 60  0001 C CNN "ventcode"
-F 5 "Optosimistorius" H 3650 2850 60  0001 C CNN "Pavadinimas"
-F 6 "0" H 4100 2550 60  0001 C CNN "Kaina"
-F 7 "SMD" H 3750 2550 60  0001 C CNN "Korpuso tipas"
-F 8 "MOC3060S" H 2450 2924 47  0001 C CNN "Gamintojo kodas"
 	1    2450 2700
 	1    0    0    -1
@@
 F 2 "" H 4450 3200 60  0001 C CNN
 F 3 "" H 1650 3650 60  0001 C CNN
-F 4 "-" H 3250 3050 60  0001 C CNN "ventcode"
-F 5 "470R" H 4200 3300 59  0001 C CNN "Nominalas"
-F 6 "0.001" H 4400 3000 60  0001 C CNN "Kaina"
-F 7 "1206" H 4450 3100 60  0001 C CNN "Korpusas"
-F 8 "1" H 4150 3000 60  0001 C CNN "Aukstis"
-F 9 "-" H 4100 2900 60  0001 C CNN "Marke"
-F 10 "Rezistorius" H 4300 3400 60  0001 C CNN "Pavadinimas"
-F 11 "-" H 4200 2900 60  0001 C CNN "Gamintojo Kodas"
-F 12 "-" H 4300 2900 60  0001 C CNN "Nuoroda"
-F 13 "SMD" H 4150 3100 60  0001 C CNN "Korpuso tipas"
-F 14 "-" H 4400 2900 60  0001 C CNN "Parametras"
-F 15 "-" H 4500 2900 60  0001 C CNN "Komentaras"
 	1    3250 3150
 	1    0    0    -1
@@
 F 2 "" H 4250 1950 50  0001 C CNN
 F 3 "" H 5000 1550 50  0001 C CNN
-F 4 "ZAJ023" H 3350 1850 60  0001 C CNN "ventcode"
-F 5 "-" H 3850 1850 60  0001 C CNN "Nominalas"
-F 6 "0" H 4750 1850 60  0001 C CNN "Kaina"
-F 7 "-" H 3950 1850 60  0001 C CNN "Korpusas"
-F 8 "10" H 4600 1850 60  0001 C CNN "Aukstis"
-F 9 "-" H 4050 1850 60  0001 C CNN "Marke"
-F 10 "Kontaktas" H 4000 2000 60  0001 C CNN "Pavadinimas"
-F 11 "-" H 4150 1850 60  0001 C CNN "Gamintojo Kodas"
-F 12 "-" H 4250 1850 60  0001 C CNN "Nuoroda"
-F 13 "DIP" H 4900 1850 60  0001 C CNN "Korpuso tipas"
-F 14 "-" H 4350 1850 60  0001 C CNN "Parametras"
-F 15 "-" H 4450 1850 60  0001 C CNN "Komentaras"
 	1    3600 1950
 	-1   0    0    1
@@
 F 2 "" H 4250 2600 50  0001 C CNN
 F 3 "" H 5000 2200 50  0001 C CNN
-F 4 "ZAJ023" H 3350 2500 60  0001 C CNN "ventcode"
-F 5 "-" H 3850 2500 60  0001 C CNN "Nominalas"
-F 6 "0" H 4750 2500 60  0001 C CNN "Kaina"
-F 7 "-" H 3950 2500 60  0001 C CNN "Korpusas"
-F 8 "10" H 4600 2500 60  0001 C CNN "Aukstis"
-F 9 "-" H 4050 2500 60  0001 C CNN "Marke"
-F 10 "Kontaktas" H 4000 2650 60  0001 C CNN "Pavadinimas"
-F 11 "-" H 4150 2500 60  0001 C CNN "Gamintojo Kodas"
-F 12 "-" H 4250 2500 60  0001 C CNN "Nuoroda"
-F 13 "DIP" H 4900 2500 60  0001 C CNN "Korpuso tipas"
-F 14 "-" H 4350 2500 60  0001 C CNN "Parametras"
-F 15 "-" H 4450 2500 60  0001 C CNN "Komentaras"
 	1    3600 2600
 	-1   0    0    1
@@
 F 2 "" H 4250 3150 50  0001 C CNN
 F 3 "" H 5000 2750 50  0001 C CNN
-F 4 "ZAJ023" H 3350 3050 60  0001 C CNN "ventcode"
-F 5 "-" H 3850 3050 60  0001 C CNN "Nominalas"
-F 6 "0" H 4750 3050 60  0001 C CNN "Kaina"
-F 7 "-" H 3950 3050 60  0001 C CNN "Korpusas"
-F 8 "10" H 4600 3050 60  0001 C CNN "Aukstis"
-F 9 "-" H 4050 3050 60  0001 C CNN "Marke"
-F 10 "Kontaktas" H 4000 3200 60  0001 C CNN "Pavadinimas"
-F 11 "-" H 4150 3050 60  0001 C CNN "Gamintojo Kodas"
-F 12 "-" H 4250 3050 60  0001 C CNN "Nuoroda"
-F 13 "DIP" H 4900 3050 60  0001 C CNN "Korpuso tipas"
-F 14 "-" H 4350 3050 60  0001 C CNN "Parametras"
-F 15 "-" H 4450 3050 60  0001 C CNN "Komentaras"
 	1    3600 3150
 	-1   0    0    1
@@
 F 2 "" H 3300 4550 50  0001 L CIN
 F 3 "http://datasheet.octopart.com/MOC3063SR2M-Fairchild-Semiconductor-datasheet-10497244.pdf" H 3300 4450 50  0001 L CNN
-F 4 "-" H 2450 4100 60  0001 C CNN "ventcode"
-F 5 "Optosimistorius" H 3650 4650 60  0001 C CNN "Pavadinimas"
-F 6 "0" H 4100 4350 60  0001 C CNN "Kaina"
-F 7 "SMD" H 3750 4350 60  0001 C CNN "Korpuso tipas"
-F 8 "MOC3060S" H 2450 4724 47  0001 C CNN "Gamintojo kodas"
 	1    2450 4500
 	1    0    0    -1
@@
 F 2 "" H 4450 4450 60  0001 C CNN
 F 3 "" H 1650 4900 60  0001 C CNN
-F 4 "-" H 3250 4300 60  0001 C CNN "ventcode"
-F 5 "470R" H 4200 4550 59  0001 C CNN "Nominalas"
-F 6 "0.001" H 4400 4250 60  0001 C CNN "Kaina"
-F 7 "1206" H 4450 4350 60  0001 C CNN "Korpusas"
-F 8 "1" H 4150 4250 60  0001 C CNN "Aukstis"
-F 9 "-" H 4100 4150 60  0001 C CNN "Marke"
-F 10 "Rezistorius" H 4300 4650 60  0001 C CNN "Pavadinimas"
-F 11 "-" H 4200 4150 60  0001 C CNN "Gamintojo Kodas"
-F 12 "-" H 4300 4150 60  0001 C CNN "Nuoroda"
-F 13 "SMD" H 4150 4350 60  0001 C CNN "Korpuso tipas"
-F 14 "-" H 4400 4150 60  0001 C CNN "Parametras"
-F 15 "-" H 4500 4150 60  0001 C CNN "Komentaras"
 	1    3250 4400
 	1    0    0    -1
@@
 F 2 "" H 4250 4050 50  0001 C CNN
 F 3 "" H 5000 3650 50  0001 C CNN
-F 4 "ZAJ023" H 3350 3950 60  0001 C CNN "ventcode"
-F 5 "-" H 3850 3950 60  0001 C CNN "Nominalas"
-F 6 "0" H 4750 3950 60  0001 C CNN "Kaina"
-F 7 "-" H 3950 3950 60  0001 C CNN "Korpusas"
-F 8 "10" H 4600 3950 60  0001 C CNN "Aukstis"
-F 9 "-" H 4050 3950 60  0001 C CNN "Marke"
-F 10 "Kontaktas" H 4000 4100 60  0001 C CNN "Pavadinimas"
-F 11 "-" H 4150 3950 60  0001 C CNN "Gamintojo Kodas"
-F 12 "-" H 4250 3950 60  0001 C CNN "Nuoroda"
-F 13 "DIP" H 4900 3950 60  0001 C CNN "Korpuso tipas"
-F 14 "-" H 4350 3950 60  0001 C CNN "Parametras"
-F 15 "-" H 4450 3950 60  0001 C CNN "Komentaras"
 	1    3600 4050
 	-1   0    0    1
@@
 F 2 "" H 4250 5000 50  0001 C CNN
 F 3 "" H 5000 4600 50  0001 C CNN
-F 4 "ZAJ023" H 3350 4900 60  0001 C CNN "ventcode"
-F 5 "-" H 3850 4900 60  0001 C CNN "Nominalas"
-F 6 "0" H 4750 4900 60  0001 C CNN "Kaina"
-F 7 "-" H 3950 4900 60  0001 C CNN "Korpusas"
-F 8 "10" H 4600 4900 60  0001 C CNN "Aukstis"
-F 9 "-" H 4050 4900 60  0001 C CNN "Marke"
-F 10 "Kontaktas" H 4000 5050 60  0001 C CNN "Pavadinimas"
-F 11 "-" H 4150 4900 60  0001 C CNN "Gamintojo Kodas"
-F 12 "-" H 4250 4900 60  0001 C CNN "Nuoroda"
-F 13 "DIP" H 4900 4900 60  0001 C CNN "Korpuso tipas"
-F 14 "-" H 4350 4900 60  0001 C CNN "Parametras"
-F 15 "-" H 4450 4900 60  0001 C CNN "Komentaras"
 	1    3600 5000
 	-1   0    0    1
@@
 F 2 "" H 4250 4600 50  0001 C CNN
 F 3 "" H 5000 4200 50  0001 C CNN
-F 4 "ZAJ023" H 3350 4500 60  0001 C CNN "ventcode"
-F 5 "-" H 3850 4500 60  0001 C CNN "Nominalas"
-F 6 "0" H 4750 4500 60  0001 C CNN "Kaina"
-F 7 "-" H 3950 4500 60  0001 C CNN "Korpusas"
-F 8 "10" H 4600 4500 60  0001 C CNN "Aukstis"
-F 9 "-" H 4050 4500 60  0001 C CNN "Marke"
-F 10 "Kontaktas" H 4000 4650 60  0001 C CNN "Pavadinimas"
-F 11 "-" H 4150 4500 60  0001 C CNN "Gamintojo Kodas"
-F 12 "-" H 4250 4500 60  0001 C CNN "Nuoroda"
-F 13 "DIP" H 4900 4500 60  0001 C CNN "Korpuso tipas"
-F 14 "-" H 4350 4500 60  0001 C CNN "Parametras"
-F 15 "-" H 4450 4500 60  0001 C CNN "Komentaras"
 	1    3600 4600
 	-1   0    0    1
